File: Three_Phase_Inverter/Three_Phase_Inverter.kicad_pcb (KiCad board)
At the start: 2 copper layers, 62.5 x 123 mm, 47 parts, among them J5 POWER, J6 OLED Display pins, Q2 IRLZ44N, Q3 IRLZ44N, Q4 IRLZ44N, Q5 IRLZ44N, Q6 IRLZ44N

Commit message: Changes made?
Parts:
- added R24: 10k, Resistor_THT:R_Axial_DIN0204_L3.6mm_D1.6mm_P7.62mm_Horizontal, F.Cu at (90.9, 99.6)
- added R25: 20k, Resistor_THT:R_Axial_DIN0204_L3.6mm_D1.6mm_P7.62mm_Horizontal, F.Cu at (90.9, 102.7)
- added R26: 10k, Resistor_THT:R_Axial_DIN0204_L3.6mm_D1.6mm_P7.62mm_Horizontal, F.Cu at (90.9, 105.9)
- added R27: 10k, Resistor_THT:R_Axial_DIN0204_L3.6mm_D1.6mm_P7.62mm_Horizontal, F.Cu at (90.9, 109.0)
- added R28: 20k, Resistor_THT:R_Axial_DIN0204_L3.6mm_D1.6mm_P7.62mm_Horizontal, F.Cu at (90.9, 112.2)
- added R29: 20k, Resistor_THT:R_Axial_DIN0204_L3.6mm_D1.6mm_P7.62mm_Horizontal, F.Cu at (90.9, 115.3)
- renumbered C100u to C1, C100n to C2, C100u to C3, C100n to C4, Vout to J3, IRLZ44N to Q1, R1k to R1, R1k to R10, R1k to R11, R300 to R12, R1k to R13, R300 to R14, R1k to R15, R300 to R16, R1k to R17, R300 to R18, R1k to R19, R1k to R2, R300 to R20, R1k to R21, R300 to R22, R1k to R23, R1k to R3, R91k to R4, R10k to R5, R1k to R6, R1k to R7, R1k to R8, R1k to R9, L7805 to U1, PC817 to U2, PC817 to U3, PC817 to U4, PC817 to U5, PC817 to U6, PC817 to U7, ESP32 to U8
Connections:
- Forward1 pad 1: GPIO27 -> Net-(Forward1-Pad1)
- R1 pad 1: GPIO25 -> Net-(R1-Pad1)
- R2 pad 1: GPIO26 -> Net-(R2-Pad1)
- R3 pad 1: GPIO27 -> Net-(Forward1-Pad1)
- Reverse1 pad 1: GPIO26 -> Net-(R2-Pad1)
- Stop1 pad 1: GPIO25 -> Net-(R1-Pad1)
- U8 pad 1: EN -> GND
- U8 pad 10: GPIO27 -> GPIO25
- U8 pad 11: GPIO14 -> GPIO26
- U8 pad 12: GPIO12* -> GPIO27
- U8 pad 13: GPIO13* -> GPIO14
- U8 pad 14: GND -> GPIO12*
- U8 pad 15: 5V -> GND
- U8 pad 16: 3.3V -> GPIO13*
- U8 pad 17: GND -> unconnected-(U8-SHD/SD2-Pad17)
- U8 pad 18: (no net) -> unconnected-(U8-SWP/SD3-Pad18)
- U8 pad 19: (no net) -> unconnected-(U8-SCS/CMD-Pad19)
- U8 pad 2: GPIO36* -> 5V
- U8 pad 20: GPIO4* -> unconnected-(U8-SCK/CLK-Pad20)
- U8 pad 21: (no net) -> unconnected-(U8-SDO/SD0-Pad21)
- U8 pad 22: (no net) -> unconnected-(U8-SDI/SD1-Pad22)
- U8 pad 23: GPIO5* -> unconnected-(U8-IO15-Pad23)
- U8 pad 25: (no net) -> unconnected-(U8-IO0-Pad25)
- U8 pad 26: GPIO21(SDA) -> GPIO4*
- U8 pad 29: GPIO22(SCL) -> GPIO5*
- U8 pad 3: (no net) -> unconnected-(U8-EN-Pad3)
- U8 pad 30: (no net) -> unconnected-(U8-IO18-Pad30)
- U8 pad 4: (no net) -> GPIO36*
- U8 pad 5: GPIO35 -> unconnected-(U8-SENSOR_VN-Pad5)
- U8 pad 6: GPIO32* -> unconnected-(U8-IO34-Pad6)
- U8 pad 7: GPIO33 -> GPIO35
- U8 pad 8: GPIO25 -> GPIO32*
- U8 pad 9: GPIO26 -> GPIO33
Routing:
- net GPIO27: track 132.2 -> 0.00 mm
- net GPIO33: track 0.00 -> 114.2 mm
- net GPIO26: track 114.2 -> 0.00 mm
- net GPIO32*: track 35.7 -> 146.0 mm
- net GPIO25: track 110.3 -> 132.2 mm

Commit message: changes
Parts:
- removed R1, R2, R3: 1k, Resistor_THT:R_Axial_DIN0204_L3.6mm_D1.6mm_P7.62mm_Horizontal
- R10, R11, R12, R13, R14, R15, R16, R17, R18, R19, R20, R21, R22, R23, R24, R25, R26, R27, R28, R29, R4, R5, R6, R7, R8, R9: footprint Resistor_THT:R_Axial_DIN0204_L3.6mm_D1.6mm_P7.62mm_Horizontal -> Resistor_THT:R_Axial_DIN0207_L6.3mm_D2.5mm_P10.16mm_Horizontal
- moved AC 104.5 mm to (198.8, 74.8), turned to 180 degrees
- moved R23 102.0 mm to (235.9, 92.8), turned to 180 degrees
- moved Q6 97.7 mm to (233.7, 84.3), turned to 180 degrees
- moved R20 84.7 mm to (226.6, 106.7), turned to 90 degrees
- moved R11 83.6 mm to (222.9, 111.6), turned to 180 degrees
- moved R21 77.7 mm to (218.7, 92.8), turned to 180 degrees
- moved U7 74.7 mm to (218.5, 106.4), turned to 90 degrees
- moved J6 73.6 mm to (197.3, 131.3), turned to 180 degrees
- moved Q5 71.6 mm to (215.2, 84.3), turned to 180 degrees
- moved R22 67.9 mm to (212.9, 106.6), turned to 90 degrees
- moved R25 67.0 mm to (143.5, 144.3), turned to 180 degrees
- moved R10 66.6 mm to (208.2, 111.4), turned to 180 degrees
- moved U8 62.2 mm to (153.2, 143.0), turned to 90 degrees
- moved R28 59.0 mm to (143.5, 138.9), turned to 180 degrees
- moved U6 58.7 mm to (204.8, 106.1), turned to 90 degrees
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- renumbered J5 to 12v, J3 to AC
Routing:
- net GPIO33: track 114.2 -> 0.00 mm
- net GPIO32*: track 146.0 -> 62.6 mm
- net GPIO27: track 0.00 -> 79.4 mm
- net GPIO25: track 132.2 -> 59.4 mm
- net GPIO26: track 0.00 -> 69.9 mm
- net GND: track 366.4 -> 421.5 mm
- net Net-(J3-Pin_2): track 86.4 -> 31.3 mm, vias 0 -> 1
- net Net-(J3-Pin_1): track 118.6 -> 69.5 mm
- net Net-(Q6-G): track 59.7 -> 26.1 mm
- net GPIO4*: track 55.4 -> 28.3 mm, vias 2 -> 0
- net GPIO21(SDA): track 57.3 -> 84.2 mm
- net GPIO35: track 38.6 -> 62.2 mm
- net 3.3V: track 21.5 -> 0.00 mm
- net GPIO5*: track 30.6 -> 9.75 mm
- net Net-(R26-Pad1): track 0.00 -> 19.9 mm
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Other:
- board size 62.5 x 123 mm -> 122.9 x 85.9 mm

Commit message: Mde Gerber, updated PCB
Parts:
- removed U4, U5, U6, U7: PC817, Package_DIP:DIP-4_W7.62mm
- R10, R11, R6, R7, R8, R9: value 1k -> 460
- U2: value PC817 -> PC847; footprint Package_DIP:DIP-4_W7.62mm -> Package_DIP:DIP-16_W7.62mm
- U3: value PC817 -> PC827; footprint Package_DIP:DIP-4_W7.62mm -> Package_DIP:DIP-8_W7.62mm
- moved U3 39.9 mm to (203.7, 106.2)
- moved R12 21.4 mm to (179.7, 107.4)
- moved C3 19.8 mm to (134.0, 111.3)
- moved C4 19.8 mm to (127.5, 111.3)
- moved R14 14.6 mm to (186.5, 107.4)
- moved J6 11.6 mm to (208.8, 133.0)
- moved R16 7.25 mm to (192.8, 107.4)
- moved R22 5.33 mm to (218.2, 107.4)
- moved U2 3.25 mm to (153.4, 106.2)
- moved R18 1.31 mm to (198.5, 107.4)
- moved R20 1.05 mm to (225.8, 107.4)
- renumbered AC to J3, 12v to J5
Connections:
- U2 pad 3: Net-(R12-Pad1) -> Net-(R7-Pad1)
- U2 pad 4: +BATT -> GND
- U3 pad 1: Net-(R7-Pad1) -> Net-(R10-Pad1)
- U3 pad 3: Net-(R14-Pad1) -> Net-(R11-Pad1)
- U3 pad 4: +BATT -> GND
- U8 pad : (no net) -> 3.3V
Routing:
- net GND: track 421.5 -> 323.2 mm
- net 3.3V: track 0.00 -> 40.5 mm
- net GPIO21(SDA): track 84.2 -> 58.0 mm
- net Net-(Q1-G): track 28.4 -> 50.8 mm
- net Net-(R18-Pad1): track 10.5 -> 31.2 mm
- net Net-(R9-Pad1): track 6.52 -> 27.0 mm
- net Net-(R16-Pad1): track 10.4 -> 30.4 mm
- net Net-(R14-Pad1): track 11.6 -> 29.2 mm, vias 1 -> 0
- net Net-(R12-Pad1): track 10.8 -> 27.4 mm, vias 1 -> 0
- net Net-(Q2-G): track 26.2 -> 39.4 mm
- net Net-(R8-Pad1): track 5.86 -> 17.9 mm
- net GPIO32*: track 62.6 -> 72.4 mm
- net Net-(R11-Pad1): track 7.06 -> 16.3 mm
- net Net-(Q3-G): track 23.4 -> 30.6 mm, vias 2 -> 0
- net Net-(Q6-G): track 26.1 -> 21.2 mm
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Other:
- board text added: "AC"
- board text added: "DC"
