File: Three_Phase_Inverter/Three_Phase_Inverter.kicad_sch (KiCad schematic)
At the start: 47 parts, among them J3 3 phase output, J5 POWER, J6 OLED Display pins, Q1 IRLZ44N, Q2 IRLZ44N, Q3 IRLZ44N, Q4 IRLZ44N, Q5 IRLZ44N, Q6 IRLZ44N, U1 L7805, U2 PC817, U3 PC817, U4 PC817, U5 PC817, U6 PC817, U7 PC817, U8 ESP32-WROOM-32

Commit message: Changes made?
Parts:
- added R24, R26, R27: 10k, Resistor_THT:R_Axial_DIN0204_L3.6mm_D1.6mm_P7.62mm_Horizontal, symbol Device:R
- added R25, R28, R29: 20k, Resistor_THT:R_Axial_DIN0204_L3.6mm_D1.6mm_P7.62mm_Horizontal, symbol Device:R
Connections:
- net GND: now also R25.2, R28.2, R29.2
- net GPIO25: now also R25.1, R26.2; no longer R1.1, Stop1.1
- net GPIO26: now also R24.2, R28.1; no longer R2.1, Reverse1.1
- net GPIO27: now also R27.2, R29.1; no longer Forward1.1, R3.1
- net EN: no longer names the net of U8.3 (EN)
- new net: Forward1.1, R27.1, R3.1
- new net: R2.1, R24.1, Reverse1.1
- new net: R1.1, R26.1, Stop1.1
Other:
- note added: "Gate driver and switching circuit"
- moved on the sheet: Forward1, R1, R3, Stop1

Commit message: changes
Parts:
- removed R1, R2, R3: 1k, Resistor_THT:R_Axial_DIN0204_L3.6mm_D1.6mm_P7.62mm_Horizontal, symbol Device:R
- R10, R11, R12, R13, R14, R15, R16, R17, R18, R19, R20, R21, R22, R23, R24, R25, R26, R27, R28, R29, R4, R5, R6, R7, R8, R9: footprint Resistor_THT:R_Axial_DIN0204_L3.6mm_D1.6mm_P7.62mm_Horizontal -> Resistor_THT:R_Axial_DIN0207_L6.3mm_D2.5mm_P10.16mm_Horizontal
Connections:
- no-connect marks 17 -> 18
Other:
- moved on the sheet: R24, R26, R27

Commit message: Mde Gerber, updated PCB
Parts:
- removed U2, U3, U4, U5, U6, U7: PC817, Package_DIP:DIP-4_W7.62mm, symbol Isolator:PC817
- added U2: PC847, Package_DIP:DIP-16_W7.62mm, symbol Isolator:PC847
- added U3: PC827, Package_DIP:DIP-8_W7.62mm, symbol Isolator:PC827
- R10, R11, R6, R7, R8, R9: value 1k -> 460
Connections:
- net +BATT: now also U2.10, U2.12, U2.14, U2.16, U3.6, U3.8
- net GND: now also U2.2, U2.4, U2.6, U2.8, U3.2, U3.4
- net at R18.1: now also U2.9
- net at R10.1: now also U3.1
- net at R6.1: now also U2.1
- net at R12.1: now also U2.15
- net at R9.1: now also U2.7
- net at R8.1: now also U2.5
- net at R20.1: now also U3.7
- net at R16.1: now also U2.11
- net at R22.1: now also U3.5
- net at R14.1: now also U2.13
- net at R11.1: now also U3.3
- net at R7.1: now also U2.3

Commit message: ~
Parts:
- Forward1, Reverse1, Stop1: value ~ -> (none)
